File: active projects/Kedi Savar/Electrical/KediSavar/KediSavar.kicad_pcb (KiCad board)
At the start: 2 copper layers, 100 x 100 mm, 76 parts, among them J1 Screw_Terminal_01x10, J2 Conn_02x20_Odd_Even, Q1 AO3400A, Q2 AO3400A, Q3 AO3400A, U1 TS3552CS, U2 TS3552CS, U3 ULN2003A, U4 ULN2003A

Commit message: Daily backup: 2026-08-04-17-23-54
Parts:
- added BATT: TestPoint, TestPoint:TestPoint_Pad_1.5x1.5mm, F.Cu at (177.6, 93.2)
- added C14: 10uF / 35-50v, Capacitor_SMD:C_1206_3216Metric_Pad1.33x1.80mm_HandSolder, F.Cu at (171.9, 135.1)
- added C18: 10uF / 35-50v, Capacitor_SMD:C_1206_3216Metric_Pad1.33x1.80mm_HandSolder, F.Cu at (181.3, 146.3)
- added D4: SS14, Diode_SMD:D_3220_8050Metric_Pad2.65x5.15mm_HandSolder, F.Cu at (105.5, 130.4)
- added D5: LED, LED_SMD:LED_0805_2012Metric_Pad1.15x1.40mm_HandSolder, F.Cu at (182.3, 93.3)
- added D6: LED, LED_SMD:LED_0805_2012Metric_Pad1.15x1.40mm_HandSolder, F.Cu at (182.3, 97.2)
- added D7: LED, LED_SMD:LED_0805_2012Metric_Pad1.15x1.40mm_HandSolder, F.Cu at (182.3, 101.0)
- added GND: TestPoint, TestPoint:TestPoint_Pad_1.5x1.5mm, F.Cu at (177.6, 104.7)
- added PWR: TestPoint, TestPoint:TestPoint_Pad_1.5x1.5mm, F.Cu at (177.6, 97.1)
- added R27: 470, Resistor_SMD:R_0805_2012Metric_Pad1.20x1.40mm_HandSolder, F.Cu at (114.1, 115.7)
- added R42: 1k, Resistor_SMD:R_0805_2012Metric_Pad1.20x1.40mm_HandSolder, F.Cu at (188.2, 93.3)
- added R43: 330, Resistor_SMD:R_0805_2012Metric_Pad1.20x1.40mm_HandSolder, F.Cu at (188.2, 97.1)
- added R44: 330, Resistor_SMD:R_0805_2012Metric_Pad1.20x1.40mm_HandSolder, F.Cu at (188.1, 101.0)
- added REF**: didoe, Can foot:didoe, F.Cu at (104.2, 127.0)
- added REF**: Fiducial_0.5mm_Mask2mm, Fiducial:Fiducial_0.5mm_Mask2mm, F.Cu at (197.1, 136.6)
- added REF**: Fiducial_0.5mm_Mask2mm, Fiducial:Fiducial_0.5mm_Mask2mm, B.Cu at (105.9, 134.7)
- added REF**: Fiducial_0.5mm_Mask2mm, Fiducial:Fiducial_0.5mm_Mask2mm, B.Cu at (194.4, 137.3)
- added REF**: Fiducial_0.5mm_Mask2mm, Fiducial:Fiducial_0.5mm_Mask2mm, B.Cu at (161.3, 65.5)
- added REF**: didoe, Can foot:didoe, F.Cu at (151.3, 113.0)
- added REF**: Fiducial_0.5mm_Mask2mm, Fiducial:Fiducial_0.5mm_Mask2mm, F.Cu at (114.0, 55.2)
- added REF**: didoe, Can foot:didoe, F.Cu at (126.8, 113.1)
- added REF**: didoe, Can foot:didoe, F.Cu at (138.7, 113.1)
- added REF**: Fiducial_0.5mm_Mask2mm, Fiducial:Fiducial_0.5mm_Mask2mm, F.Cu at (196.5, 63.0)
- added U3: AQY212GZS, Package_SO:SO-4_4.4x4.3mm_P2.54mm, F.Cu at (109.2, 120.7)
- added uC: TestPoint, TestPoint:TestPoint_Pad_1.5x1.5mm, F.Cu at (177.6, 100.9)
- J2: renamed from J1; footprint Can foot:wago 256 410 -> Can foot:Wago 256 410
- moved U5 168.0 mm to (186.9, 135.8), turned to 90 degrees
- moved U4 151.8 mm to (170.5, 127.6), turned to 90 degrees
- moved C13 143.2 mm to (191.8, 129.3), turned to 180 degrees
- moved C19 139.5 mm to (186.4, 148.2)
- moved C12 134.9 mm to (183.5, 129.3)
- moved C8 132.0 mm to (188.0, 85.7), turned to 180 degrees
- moved R35 128.6 mm to (198.1, 124.5)
- moved R39 128.4 mm to (198.1, 129.3), turned to 180 degrees
- moved C11 123.3 mm to (176.7, 124.9), turned to 180 degrees
- moved R34 122.1 mm to (191.8, 124.4)
- moved C17 121.5 mm to (169.8, 142.8)
- moved C10 120.0 mm to (167.3, 120.3)
- moved U2 119.1 mm to (148.7, 93.8)
- moved C16 118.7 mm to (181.3, 142.5), turned to 180 degrees
- moved C9 114.2 mm to (170.2, 95.5)
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- renumbered C17 to C1, C8 to C10, C9 to C11, C3 to C12, C4 to C13, C6 to C15, C1 to C16, C7 to C17, C2 to C19, C16 to C2, C15 to C3, C14 to C4, C13 to C5, C12 to C6, C11 to C7, C5 to C8, C10 to C9, D3 to D1, D1 to D3, J2 to J1, L2 to L1, L1 to L2, Q3 to Q1, Q1 to Q3, R15 to R1, R22 to R10, R10 to R11, R23 to R12, R9 to R13, R24 to R14, R25 to R15, R33 to R16, R26 to R17, R34 to R18, R27 to R19, R18 to R2, R35 to R20, R28 to R21, R36 to R22, R29 to R23, R37 to R24, R30 to R25, R38 to R26, R6 to R28, R8 to R29, R14 to R3, R5 to R30, R17 to R31, R40 to R32, R32 to R33, R2 to R34, R4 to R35, R39 to R36, R31 to R37, R16 to R38, R3 to R39, R19 to R4, R7 to R40, R1 to R41, R13 to R5, R20 to R6, R12 to R7, R21 to R8, R11 to R9, U3 to U1, U4 to U2, U2 to U4, U1 to U5
Connections:
- A1 pad 15: SW_3r -> SW_5r
- A1 pad 16: SW_2r -> SW_6r
- A1 pad 17: SW_1r -> SW_7r
- A1 pad 18: LED_4p -> LED_1p
- A1 pad 3: LED_2p -> LED_3p
- A1 pad 35: CTL_Gr -> CTL_Bz
- A1 pad 36: CTL_Gl -> CTL_Gr
- A1 pad 37: CTL_Bz -> CTL_Gl
- A1 pad 38: unconnected-(A1-Pad38) -> CTL_SENS
- A1 pad 4: SW_7r -> SW_1r
- A1 pad 46: LED_1p -> LED_4p
- A1 pad 5: SW_6r -> SW_2r
- A1 pad 6: SW_5r -> SW_3r
- A1 pad 8: LED_3p -> LED_2p
- J1 pad 33: LED_Ac -> LED_DpC
- J1 pad 34: LED_DpC -> LED_Ac
- J1 pad 35: LED_Bc -> LED_Gc
- J1 pad 36: LED_Gc -> LED_Bc
- J1 pad 37: LED_Cc -> LED_Fc
- J1 pad 38: LED_Fc -> LED_Cc
- J1 pad 39: LED_Dc -> LED_Ec
- J1 pad 40: LED_Ec -> LED_Dc
- J2 pad 4: Gr_c -> Gl_c
- J2 pad 5: Gl_c -> Gr_c
- J2 pad 7: 16v_BATT -> 16v_BATT_Sens
Routing:
- net 5v_uC: track 0.00 -> 330.2 mm, vias 0 -> 2
- net 5v_PWR: track 0.00 -> 314.2 mm, vias 0 -> 7
- net 16v_BATT: track 0.00 -> 250.4 mm, vias 0 -> 3
- net CTL_Gl: track 0.00 -> 144.0 mm, vias 0 -> 1
- net CTL_Gr: track 0.00 -> 134.6 mm, vias 0 -> 1
- net CTL_Bz: track 0.00 -> 131.5 mm, vias 0 -> 1
- net GND: track 0.00 -> 111.8 mm, vias 0 -> 13
- net SW_3v3: track 0.00 -> 95.2 mm
- net CTL_PWR: track 0.00 -> 93.1 mm, vias 0 -> 1
- net CTL_SENS: track 0.00 -> 91.0 mm, vias 0 -> 4
- net LED_Fp: track 0.00 -> 82.0 mm, vias 0 -> 2
- net LED_Gp: track 0.00 -> 80.8 mm, vias 0 -> 2
- net LED_Dpp: track 0.00 -> 79.2 mm, vias 0 -> 2
- net 16v_BATT_Sens: track 0.00 -> 70.6 mm
- net RLY_TRIG: track 0.00 -> 59.5 mm, vias 0 -> 1
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- added copper zone on B.Cu, net GND
- added copper zone on F.Cu, net GND
Other:
- board text added: "1-PWR"
- board text added: "2-PWR"
- board text added: "3-PWR"
- board text added: "4-GL"
- board text added: "5-GR"
- board text added: "6-BZ"
- board text added: "7-BATT"
- board text added: "BATT"
- board text added: "BOTTOM"
- board text added: "GND"
- board text added: "Kedi Savar v1.0"
