File: active projects/Kedi Savar/Electrical/KediSavar/KediSavar.kicad_sch (KiCad schematic)
At the start: 72 parts, among them J1 Screw_Terminal_01x10, J2 Conn_02x20_Odd_Even, Q1 AO3400A, Q2 AO3400A, Q3 AO3400A, U1 TS3552CS, U2 TS3552CS, U3 ULN2003A, U4 ULN2003A

Commit message: Daily backup: 2026-08-04-17-23-54
Parts:
- added C14, C18: 10uF / 35-50v, Capacitor_SMD:C_1206_3216Metric_Pad1.33x1.80mm_HandSolder, symbol Device:C
- added D4: SS14, Diode_SMD:D_3220_8050Metric_Pad2.65x5.15mm_HandSolder, symbol Device:D
- added D5, D6, D7: LED, LED_SMD:LED_0805_2012Metric_Pad1.15x1.40mm_HandSolder, symbol Device:LED
- added R27: 470, Resistor_SMD:R_0805_2012Metric_Pad1.20x1.40mm_HandSolder, symbol Device:R
- added R42: 1k, Resistor_SMD:R_0805_2012Metric_Pad1.20x1.40mm_HandSolder, symbol Device:R
- added R43, R44: 330, Resistor_SMD:R_0805_2012Metric_Pad1.20x1.40mm_HandSolder, symbol Device:R
- added TP1, TP2, TP3, TP4: TestPoint, TestPoint:TestPoint_Pad_1.5x1.5mm, symbol Connector:TestPoint
- added U3: AQY212GZS, Package_SO:SO-4_4.4x4.3mm_P2.54mm, symbol Relay_SolidState:AQY282S
- A1: KiLib_Generator (none) -> connector/pin_header_socket
- C1: renamed from C17; KiLib_Generator (none) -> SMD_2terminal_chip_molded
- C10: renamed from C8; KiLib_Generator (none) -> SMD_2terminal_chip_molded
- C11: renamed from C9; KiLib_Generator (none) -> SMD_2terminal_chip_molded
- C12: renamed from C3; KiLib_Generator (none) -> SMD_2terminal_chip_molded
- C13: renamed from C4; KiLib_Generator (none) -> SMD_2terminal_chip_molded
- C15: renamed from C6; KiLib_Generator (none) -> SMD_2terminal_chip_molded
- C16: renamed from C1; KiLib_Generator (none) -> SMD_2terminal_chip_molded
- C17: renamed from C7; KiLib_Generator (none) -> SMD_2terminal_chip_molded
- C19: renamed from C2; KiLib_Generator (none) -> SMD_2terminal_chip_molded
- C2: renamed from C16; KiLib_Generator (none) -> SMD_2terminal_chip_molded
- C3: renamed from C15; KiLib_Generator (none) -> SMD_2terminal_chip_molded
- C4: renamed from C14; KiLib_Generator (none) -> SMD_2terminal_chip_molded
- C5: renamed from C13; KiLib_Generator (none) -> SMD_2terminal_chip_molded
- C6: renamed from C12; KiLib_Generator (none) -> SMD_2terminal_chip_molded
- C7: renamed from C11; KiLib_Generator (none) -> SMD_2terminal_chip_molded
- C8: renamed from C5; KiLib_Generator (none) -> SMD_2terminal_chip_molded
- C9: renamed from C10; KiLib_Generator (none) -> SMD_2terminal_chip_molded
- D1: renamed from D3; KiLib_Generator (none) -> SMD_2terminal_chip_molded
- D2: KiLib_Generator (none) -> SMD_2terminal_chip_molded
- D3: renamed from D1; KiLib_Generator (none) -> SMD_2terminal_chip_molded
- J1: renamed from J2; KiLib_Generator (none) -> connector/pin_header_socket
- J2: renamed from J1; footprint Can foot:wago 256 410 -> Can foot:Wago 256 410
- Q1: renamed from Q3; KiLib_Generator (none) -> package/gullwing
- Q2: KiLib_Generator (none) -> package/gullwing
- Q3: renamed from Q1; KiLib_Generator (none) -> package/gullwing
- R1: renamed from R15; KiLib_Generator (none) -> SMD_2terminal_chip_molded
- R10: renamed from R22; KiLib_Generator (none) -> SMD_2terminal_chip_molded
- R11: renamed from R10; KiLib_Generator (none) -> SMD_2terminal_chip_molded
- R12: renamed from R23; KiLib_Generator (none) -> SMD_2terminal_chip_molded
- R13: renamed from R9; KiLib_Generator (none) -> SMD_2terminal_chip_molded
- R14: renamed from R24; KiLib_Generator (none) -> SMD_2terminal_chip_molded
- R15: renamed from R25; KiLib_Generator (none) -> SMD_2terminal_chip_molded
- R16: renamed from R33; KiLib_Generator (none) -> SMD_2terminal_chip_molded
- R17: renamed from R26; KiLib_Generator (none) -> SMD_2terminal_chip_molded
- R18: renamed from R34; KiLib_Generator (none) -> SMD_2terminal_chip_molded
- R19: renamed from R27; KiLib_Generator (none) -> SMD_2terminal_chip_molded
- R2: renamed from R18; KiLib_Generator (none) -> SMD_2terminal_chip_molded
- R20: renamed from R35; KiLib_Generator (none) -> SMD_2terminal_chip_molded
- R21: renamed from R28; KiLib_Generator (none) -> SMD_2terminal_chip_molded
- R22: renamed from R36; KiLib_Generator (none) -> SMD_2terminal_chip_molded
- R23: renamed from R29; KiLib_Generator (none) -> SMD_2terminal_chip_molded
- R24: renamed from R37; KiLib_Generator (none) -> SMD_2terminal_chip_molded
- R25: renamed from R30; KiLib_Generator (none) -> SMD_2terminal_chip_molded
- R26: renamed from R38; KiLib_Generator (none) -> SMD_2terminal_chip_molded
- R28: renamed from R6; KiLib_Generator (none) -> SMD_2terminal_chip_molded
- R29: renamed from R8; KiLib_Generator (none) -> SMD_2terminal_chip_molded
- R3: renamed from R14; KiLib_Generator (none) -> SMD_2terminal_chip_molded
- R30: renamed from R5; KiLib_Generator (none) -> SMD_2terminal_chip_molded
- R31: renamed from R17; KiLib_Generator (none) -> SMD_2terminal_chip_molded
- R32: renamed from R40; KiLib_Generator (none) -> SMD_2terminal_chip_molded
- R33: renamed from R32; KiLib_Generator (none) -> SMD_2terminal_chip_molded
- R34: renamed from R2; KiLib_Generator (none) -> SMD_2terminal_chip_molded
- R35: renamed from R4; KiLib_Generator (none) -> SMD_2terminal_chip_molded
- R36: renamed from R39; KiLib_Generator (none) -> SMD_2terminal_chip_molded
- R37: renamed from R31; KiLib_Generator (none) -> SMD_2terminal_chip_molded
- R38: renamed from R16; KiLib_Generator (none) -> SMD_2terminal_chip_molded
- R39: renamed from R3; KiLib_Generator (none) -> SMD_2terminal_chip_molded
- R4: renamed from R19; KiLib_Generator (none) -> SMD_2terminal_chip_molded
- R40: renamed from R7; KiLib_Generator (none) -> SMD_2terminal_chip_molded
- R41: renamed from R1; KiLib_Generator (none) -> SMD_2terminal_chip_molded
- R5: renamed from R13; KiLib_Generator (none) -> SMD_2terminal_chip_molded
- R6: renamed from R20; KiLib_Generator (none) -> SMD_2terminal_chip_molded
- R7: renamed from R12; KiLib_Generator (none) -> SMD_2terminal_chip_molded
- R8: renamed from R21; KiLib_Generator (none) -> SMD_2terminal_chip_molded
- R9: renamed from R11; KiLib_Generator (none) -> SMD_2terminal_chip_molded
- U1: renamed from U3; KiLib_Generator (none) -> package/gullwing
- U2: renamed from U4; KiLib_Generator (none) -> package/gullwing
- U4: renamed from U2; KiLib_Generator (none) -> package/gullwing
- U5: renamed from U1; KiLib_Generator (none) -> package/gullwing
- renumbered L2 to L1, L1 to L2
Connections:
- net 16v_BATT: now also C14.1, C18.1, D4.1 (K), R42.1, U3.4; no longer J2.7 (Pin_7)
- net 5v_PWR: now also R43.1
- net 5v_uC: now also R44.1
- net CTL_Bz: now also A1.35; no longer A1.37
- net CTL_Gl: now also A1.37; no longer A1.36
- net CTL_Gr: now also A1.36; no longer A1.35
- net GND: now also C14.2, C18.2, TP4.1, U3.2
- net Gl_c: now also J2.4 (Pin_4); no longer J2.5 (Pin_5)
- net Gr_c: now also J2.5 (Pin_5); no longer J2.4 (Pin_4)
- net LED_1p: now also A1.18; no longer A1.46
- net LED_2p: now also A1.8; no longer A1.3
- net LED_3p: now also A1.3; no longer A1.8
- net LED_4p: now also A1.46; no longer A1.18
- net LED_Ac: now also J1.34 (Pin_34); no longer J1.33 (Pin_33)
- net LED_Bc: now also J1.36 (Pin_36); no longer J1.35 (Pin_35)
- net LED_Cc: now also J1.38 (Pin_38); no longer J1.37 (Pin_37)
- net LED_Dc: now also J1.40 (Pin_40); no longer J1.39 (Pin_39)
- net LED_DpC: now also J1.33 (Pin_33); no longer J1.34 (Pin_34)
- net LED_Ec: now also J1.39 (Pin_39); no longer J1.40 (Pin_40)
- net LED_Fc: now also J1.37 (Pin_37); no longer J1.38 (Pin_38)
- net LED_Gc: now also J1.35 (Pin_35); no longer J1.36 (Pin_36)
- net SW_1r: now also A1.4; no longer A1.17
- net SW_2r: now also A1.5; no longer A1.16
- net SW_3r: now also A1.6; no longer A1.15
- net SW_5r: now also A1.15; no longer A1.6
- net SW_6r: now also A1.16; no longer A1.5
- net SW_7r: now also A1.17; no longer A1.4
- net CTL_SENS: now reaches A1.38
- net CTL_SENS: now also R27.1
- new net: D6.1 (K), TP2.1
- new net: D6.2 (A), R43.2
- new net: R27.2, U3.1
- new net: D7.1 (K), TP3.1
- new net: D5.1 (K), TP1.1
- new net: D5.2 (A), R42.2
- new net: D7.2 (A), R44.2
- new net 16v_BATT_Sens: D4.2 (A), J2.7 (Pin_7), U3.3
- no-connect marks 26 -> 25
