File: active projects/Bike Power Meter/Electronics/Bike PWR/_restore_backup_2026-08-13T09-02-38-164/Bike PWR.kicad_pcb (KiCad board)
At the start: 4 copper layers, 55 x 55 mm, 26 parts, among them J1 Batt Holder, J3 Analyzer / Flasher, J4 Bridge, U1 LSM6DSLTR, U3 ScioSense PS09

Commit message: Daily update: 2026-08-14 17:02:38
Parts:
- moved JP2 72.2 mm to (113.5, 102.2)
- moved JP1 67.6 mm to (113.5, 98.7)
- moved J4 65.6 mm to (118.2, 81.9), turned to 0 degrees
- moved U1 60.1 mm to (131.7, 99.5), turned to 0 degrees
- moved C1 56.5 mm to (121.9, 80.5), turned to 0 degrees
- moved J1 56.4 mm to (131.4, 92.4), turned to 0 degrees
- moved C2 54.2 mm to (121.9, 82.2), turned to 0 degrees
- moved U3 43.4 mm to (125.0, 94.2), turned to 0 degrees
- moved J3 18.5 mm to (140.1, 87.7), turned to 180 degrees
- moved U2 2.03 mm to (171.1, 82.0)
Connections:
- J4 pad 1: GND -> VCC_LOAD
- J4 pad 2: SG_B -> VCC_LOAD
- J4 pad 3: SG_A -> SG_A1
- J4 pad 4: GND -> SG_B1
- J4 pad 5: SG_C -> GND_HA
- J4 pad 6: SG_D -> GND_HA
- JP1 pad 2: GND -> VDD
- U3 pad 13: SG_B -> SG_B1
- U3 pad 14: SG_B -> unconnected-(U3-SG_B2-Pad14)
- U3 pad 15: SG_A -> SG_A1
- U3 pad 16: SG_A -> unconnected-(U3-SG_A2-Pad16)
- U3 pad 23: SG_C -> unconnected-(U3-SG_C2-Pad23)
- U3 pad 24: SG_C -> unconnected-(U3-SG_C1-Pad24)
- U3 pad 25: SG_D -> unconnected-(U3-SG_D2-Pad25)
- U3 pad 26: SG_D -> unconnected-(U3-SG_D1-Pad26)
Other:
- board size 55 x 55 mm -> 60 x 60 mm
