File: active projects/Bike Power Meter/Electronics/Bike PWR/_restore_backup_2026-08-20T09-16-27-464/Bike PWR.kicad_pcb (KiCad board)
At the start: 4 copper layers, 45 x 45 mm, 53 parts, among them J1 Batt Holder, J2 Bridge, J3 Analyzer / Flasher, Q1 BC857, Q2 BC857, Q3 BC857, Q4 BC857, Q5 BC857, Q6 BC857, U1 BMI160, U3 ScioSense PS09, Y1 Resonator

Commit message: Update: Bike Power Meter Electronics folder - 2026-08-20 17:21:52
Parts:
- moved Q6 36.8 mm to (118.3, 113.8)
- moved Q4 36.7 mm to (118.3, 108.6)
- moved Q5 36.6 mm to (122.9, 113.8), turned to 0 degrees
- moved Q2 36.6 mm to (118.3, 103.8)
- moved Q3 36.4 mm to (122.9, 108.7), turned to 0 degrees
- moved Q1 36.3 mm to (122.9, 103.6), turned to 0 degrees
- moved FB6 35.6 mm to (148.0, 132.3), turned to 180 degrees
- moved FB8 34.6 mm to (148.0, 135.8), turned to 180 degrees
- moved FB5 32.8 mm to (148.0, 130.6), turned to 180 degrees
- moved FB7 31.7 mm to (148.0, 134.1), turned to 180 degrees
- moved FB2 29.3 mm to (150.8, 135.8), turned to 180 degrees
- moved FB4 28.4 mm to (150.8, 139.3), turned to 180 degrees
- moved C17 28.2 mm to (153.6, 135.8), turned to 180 degrees
- moved C15 26.4 mm to (153.6, 132.3), turned to 180 degrees
- moved FB1 26.2 mm to (150.8, 134.1), turned to 180 degrees
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Connections:
- U2 pad 5: unconnected-(U2-P0.20-Pad5) -> (no net)
Routing:
- net VDD: track 97.3 -> 27.0 mm, vias 7 -> 6
- net GND: track 85.1 -> 44.1 mm, vias 19 -> 18
- net IMU_INT1: track 30.6 -> 3.09 mm, vias 2 -> 1
- net UART_TX: track 24.3 -> 0.00 mm
- net UART_RX: track 21.5 -> 0.00 mm
- net SWDIO: track 19.3 -> 0.00 mm
- net SWDCLK: track 17.5 -> 0.00 mm
- net SG_D1: track 19.0 -> 2.11 mm
- net SG_C2: track 18.7 -> 2.23 mm
- net SG_D2: track 18.1 -> 2.16 mm
- net SG_C1: track 17.5 -> 2.19 mm
- net CCOMP: track 16.1 -> 1.99 mm, vias 1 -> 0
- net RESET_MCU: track 12.3 -> 0.00 mm
- net Net-(J2-Pin_6): track 12.0 -> 0.00 mm
- net Net-(J2-Pin_7): track 12.0 -> 0.00 mm
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